File: Hardware/Pi-based PCB.kicad_pcb (KiCad board)
At the start: 2 copper layers, 56 x 65 mm, 49 parts, among them IC2 AP2205-W5-7, J1 XT60PW-M, J11 Conn_Coaxial, J2 Conn_Coaxial, J3 Conn_02x20_Odd_Even, U1 MAX-M10S, U2 RFM95W-868S2, U3 DPS368, U4 TPSM863257RDXR, U7 ICM-20608-G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

Commit message: Relabelled some of the files
Parts:
- added D1: DST1550S, Package_TO_SOT_SMD:TO-277B, F.Cu at (106.1, 95.0)
- added D4: DST1550S, Package_TO_SOT_SMD:TO-277B, F.Cu at (111.6, 95.0)
- added D5: RED_LED, LED_SMD:LED_0603_1608Metric, F.Cu at (109.3, 79.8)
- added D6: RED_LED, LED_SMD:LED_0603_1608Metric, F.Cu at (109.3, 82.4)
- added Firing1: EMERALD_LED, LED_SMD:LED_0402_1005Metric, F.Cu at (112.9, 84.7)
- added Firing2: EMERALD_LED, LED_SMD:LED_0402_1005Metric, F.Cu at (112.9, 86.7)
- added J4: Conn_01x02_Male, TerminalBlock_Phoenix:TerminalBlock_Phoenix_PT-1,5-2-3.5-H_1x02_P3.50mm_Horizontal, F.Cu at (88.0, 94.7)
- added J5: Conn_01x02_Male, TerminalBlock_Phoenix:TerminalBlock_Phoenix_PT-1,5-2-3.5-H_1x02_P3.50mm_Horizontal, F.Cu at (88.0, 106.6)
- added J6: Conn_01x02_Male, TerminalBlock_Phoenix:TerminalBlock_Phoenix_PT-1,5-2-3.5-H_1x02_P3.50mm_Horizontal, F.Cu at (97.0, 94.7)
- added R18: 120, Resistor_SMD:R_0402_1005Metric, F.Cu at (105.8, 85.5)
- added R20: 120, Resistor_SMD:R_0603_1608Metric, F.Cu at (109.2, 87.5)
- added R4: 10K, Resistor_SMD:R_0402_1005Metric, F.Cu at (105.8, 79.5)
- added R5: 120, Resistor_SMD:R_0402_1005Metric, F.Cu at (105.8, 81.5)
- added R8: 10K, Resistor_SMD:R_0402_1005Metric, F.Cu at (105.8, 83.5)
- added R9: 120, Resistor_SMD:R_0603_1608Metric, F.Cu at (109.2, 85.0)
- added U5: DRV8212P, Package_SON:WSON-8-1EP_2x2mm_P0.5mm_EP0.9x1.6mm_ThermalVias, F.Cu at (96.5, 104.4)
- added U6: LTV-247, Package_SO:SOP-16_4.4x10.4mm_P1.27mm, F.Cu at (90.0, 84.6)
- added U9: LTV-247, Package_SO:SOP-16_4.4x10.4mm_P1.27mm, F.Cu at (99.5, 84.6)
Connections:
- net /power/BB_IN renamed /DeployPWR
- net /power/LDO5.5V_IN renamed +5.5V
- J3 pad 40: unconnected-(J3-Pin_40-Pad40) -> /Nuke 1
