File: Hardware/Pi-based PCB.kicad_sch (KiCad schematic)
At the start: 4 parts, among them J3 Conn_02x20_Odd_Even

Commit message: Reorganised
Connections:
- net Nuke 1: now reaches J3.40 (Pin_40)
- no-connect marks 21 -> 20
Other:
- sheet power ports: added DeployPWR; removed 5V
- sheet pyro ports: added Nuke 1; removed none
Changed lines of the file:
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@@
-	)
-	(no_connect
-		(at 109.22 96.52)
 	)
 	(no_connect
@@
 	(wire
 		(pts
+			(xy 149.86 134.62) (xy 157.48 134.62)
+		)
+		(stroke
+			(width 0)
+			(type default)
+		)
+	)
+	(wire
+		(pts
 			(xy 144.78 104.14) (xy 156.21 104.14)
 		)
@@
 	(wire
 		(pts
+			(xy 109.22 96.52) (xy 115.57 96.52)
+		)
+		(stroke
+			(width 0)
+			(type default)
+		)
+	)
+	(wire
+		(pts
+			(xy 93.726 127) (xy 102.87 127)
+		)
+		(stroke
+			(width 0)
+			(type default)
+		)
+	)
+	(wire
+		(pts
 			(xy 109.22 93.98) (xy 115.57 93.98)
 		)
@@
 		(pts
 			(xy 147.32 50.8) (xy 158.75 50.8)
-		)
-		(stroke
-			(width 0)
-			(type default)
-		)
-	)
-	(wire
-		(pts
-			(xy 96.52 121.92) (xy 102.87 121.92)
 		)
 		(stroke
@@
 		)
 	)
+	(label "DeployPWR"
+		(at 93.726 127 180)
+		(effects
+			(font
+				(size 1.27 1.27)
+			)
+			(justify right bottom)
+		)
+	)
 	(label "PI_MISO"
 		(at 83.82 73.66 180)
@@
 		)
 	)
+	(label "Nuke 1"
+		(at 115.57 96.52 0)
+		(effects
+			(font
+				(size 1.27 1.27)
+			)
+			(justify left bottom)
+		)
+	)
+	(label "Nuke 1"
+		(at 149.86 134.62 180)
+		(effects
+			(font
+				(size 1.27 1.27)
+			)
+			(justify right bottom)
+		)
+	)
 	(label "Nuke 0"
 		(at 115.57 91.44 0)
@@
 		)
 	)
+	(label "DeployPWR"
+		(at 149.86 129.54 180)
+		(effects
+			(font
+				(size 1.27 1.27)
+			)
+			(justify right bottom)
+		)
+	)
 	(label "Cont0"
 		(at 149.86 127 180)
@@
 			)
 			(justify right bottom)
-		)
-	)
-	(hierarchical_label "5.5V"
-		(shape output)
-		(at 100.33 146.05 90)
-		(effects
-			(font
-				(size 1.27 1.27)
-			)
-			(justify left)
-		)
-	)
-	(hierarchical_label "DeployPWR"
-		(shape input)
-		(at 149.86 129.54 180)
-		(effects
-			(font
-				(size 1.27 1.27)
-			)
-			(justify right)
-		)
-	)
-	(symbol
-		(lib_id "power:+5V")
-		(at 96.52 121.92 0)
-		(unit 1)
-		(exclude_from_sim no)
-		(in_bom yes)
-		(on_board yes)
-		(dnp no)
-		(fields_autoplaced yes)
-		(property "Reference" "#PWR014"
-			(at 96.52 125.73 0)
-			(effects
-				(font
-					(size 1.27 1.27)
-				)
-				(hide yes)
-			)
-		)
-		(property "Value" "+5V"
-			(at 96.52 116.84 0)
-			(effects
-				(font
-					(size 1.27 1.27)
-				)
-			)
-		)
-		(property "Footprint" ""
-			(at 96.52 121.92 0)
-			(effects
-				(font
-					(size 1.27 1.27)
-				)
-				(hide yes)
-			)
-		)
-		(property "Datasheet" ""
-			(at 96.52 121.92 0)
-			(effects
-				(font
-					(size 1.27 1.27)
-				)
-				(hide yes)
-			)
-		)
-		(property "Description" "Power symbol creates a global label with name \"+5V\""
-			(at 96.52 121.92 0)
-			(effects
-				(font
-					(size 1.27 1.27)
-				)
-				(hide yes)
-			)
-		)
-		(pin "1"
-		)
-		(instances
-			(project ""
-				(path "/e4035b22-64c9-4a42-9837-ade8aec3882f"
-					(reference "#PWR014")
-					(unit 1)
-				)
-			)
 		)
 	)
@@
 				(path "/e4035b22-64c9-4a42-9837-ade8aec3882f"
 					(reference "TP6")
+					(unit 1)
+				)
+			)
+		)
+	)
+	(symbol
+		(lib_id "power:+5V")
+		(at 100.33 146.05 0)
+		(unit 1)
+		(exclude_from_sim no)
+		(in_bom yes)
+		(on_board yes)
+		(dnp no)
+		(fields_autoplaced yes)
+		(property "Reference" "#PWR035"
+			(at 100.33 149.86 0)
+			(effects
+				(font
+					(size 1.27 1.27)
+				)
+				(hide yes)
+			)
+		)
+		(property "Value" "+5.5V"
+			(at 100.33 140.97 0)
+			(effects
+				(font
+					(size 1.27 1.27)
+				)
+			)
+		)
+		(property "Footprint" ""
+			(at 100.33 146.05 0)
+			(effects
+				(font
+					(size 1.27 1.27)
+				)
+				(hide yes)
+			)
+		)
+		(property "Datasheet" ""
+			(at 100.33 146.05 0)
+			(effects
+				(font
+					(size 1.27 1.27)
+				)
+				(hide yes)
+			)
+		)
+		(property "Description" "Power symbol creates a global label with name \"+5V\""
+			(at 100.33 146.05 0)
+			(effects
+				(font
+					(size 1.27 1.27)
+				)
+				(hide yes)
+			)
+		)
+		(pin "1"
+		)
+		(instances
+			(project "Pi-based PCB"
+				(path "/e4035b22-64c9-4a42-9837-ade8aec3882f"
+					(reference "#PWR035")
 					(unit 1)
 				)
@@
 		)
 		(instances
-			(project ""
+			(project "Pi-based PCB"
 				(path "/e4035b22-64c9-4a42-9837-ade8aec3882f"
 					(reference "#PWR015")
@@
 		)
 		(instances
-			(project ""
+			(project "Pi-based PCB"
 				(path "/e4035b22-64c9-4a42-9837-ade8aec3882f"
 					(reference "J3")
@@
 		)
 		(instances
-			(project ""
+			(project "Pi-based PCB"
 				(path "/e4035b22-64c9-4a42-9837-ade8aec3882f"
 					(reference "#PWR023")
@@
 			)
 		)
-		(pin "5V" output
-			(at 102.87 121.92 180)
+		(pin "DeployPWR" output
+			(at 102.87 127 180)
 			(effects
 				(font
@@
 			(effects
 				(font
+					(size 1.27 1.27)
+				)
+				(justify left)
+			)
+		)
+		(pin "Nuke 1" input
+			(at 157.48 134.62 180)
+			(effects
+				(font

Commit message: Relabelled some of the files
Other:
- sheet IMU: file untitled.kicad_sch -> imu.kicad_sch
Changed lines of the file:
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@@
 			)
 		)
-		(property "Sheetfile" "untitled.kicad_sch"
+		(property "Sheetfile" "imu.kicad_sch"
 			(at 158.75 33.6046 0)
 			(effects
@@
 				)
 				(justify left top)
-				(hide yes)
 			)
 		)
