File: Hardware/pyro.kicad_sch (KiCad schematic)
At the start: 11 parts, among them J4 Conn_01x02_Male, Q1 BSZ025N04LS, U6 LTV-247

Commit message: Reorganised
Parts:
- added D2: V8PAM10S-M3/I, iclr:V8PAM10SM3I, symbol Device:D_Schottky_Small_Filled
- added D4: DST1550S, Package_TO_SOT_SMD:TO-277B, symbol Device:D_Schottky_AAK
- added D6: RED_LED, LED_SMD:LED_0603_1608Metric, symbol Device:LED
- added D7: S-102T, iclr:SODFL3516X70N, symbol iclr:S-102T
- added Firing2: EMERALD_LED, LED_SMD:LED_0402_1005Metric, symbol Device:LED
- added J6: Conn_01x02_Male, TerminalBlock_Phoenix:TerminalBlock_Phoenix_PT-1,5-2-3.5-H_1x02_P3.50mm_Horizontal, symbol Connector:Conn_01x02_Male
- added Q2: BSZ025N04LS, iclr:BSZ025N04LS, symbol iclr:BSZ025N04LS
- added R5: 120, Resistor_SMD:R_0402_1005Metric, symbol Device:R
- added R8: 10K, Resistor_SMD:R_0402_1005Metric, symbol Device:R
- added R9: 120, Resistor_SMD:R_0603_1608Metric, symbol Device:R
- added U9: LTV-247, Package_SO:SOP-16_4.4x10.4mm_P1.27mm, symbol Isolator:LTV-247
Connections:
- net +3V3: now also U9.10
- net Cont0: now also R9.1, U9.9
- net DeployPWR: now also D2.1 (K), J6.1 (Pin_1)
- net GND: now also D6.1 (K), D7.1 (K), Q2.1 (S), Q2.2 (S), Q2.3 (S), Q2.A1 (S), R5.2, R8.2
- new net: D6.2 (A), R9.2
- new net: Firing2.1 (K), R5.1
- new net: D2.2 (A), D4.1 (A), D4.2 (A), J6.2 (Pin_2), U9.7
- new net: D4.3 (K), Q2.5 (D), Q2.6 (D), Q2.7 (D), Q2.8 (D), Q2.A5 (D)
- new net: D7.2 (A), U9.8
- new net Nuke 1: Firing2.2 (A), Q2.4 (G), R8.1
Other:
- moved on the sheet: D1, D11, D16, D5, Firing1, J4, Q1, R18, R20, R4, U6D

Commit message: Modified power
Connections:
- net Cont0: no longer R9.1, U9.9
- new net Cont1: R9.1, U9.9
Changed lines of the file:
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@@
 		)
 	)
-	(hierarchical_label "Cont0"
+	(hierarchical_label "Cont1"
 		(shape output)
 		(at 157.48 121.92 180)
@@
 		)
 		(instances
-			(project "Pi-based PCB"
+			(project "Ricardo-Cappy"
 				(path "/e4035b22-64c9-4a42-9837-ade8aec3882f/6c4172b2-a587-4406-930d-3d10d9850979"
 					(reference "R9")
@@
 		)
 		(instances
-			(project "Pi-based PCB"
+			(project "Ricardo-Cappy"
 				(path "/e4035b22-64c9-4a42-9837-ade8aec3882f/6c4172b2-a587-4406-930d-3d10d9850979"
 					(reference "#PWR026")
@@
 		)
 		(instances
-			(project "Pi-based PCB"
+			(project "Ricardo-Cappy"
 				(path "/e4035b22-64c9-4a42-9837-ade8aec3882f/6c4172b2-a587-4406-930d-3d10d9850979"
 					(reference "D6")
@@
 		)
 		(instances
-			(project "Pi-based PCB"
+			(project "Ricardo-Cappy"
 				(path "/e4035b22-64c9-4a42-9837-ade8aec3882f/6c4172b2-a587-4406-930d-3d10d9850979"
 					(reference "R8")
@@
 		)
 		(instances
-			(project "Pi-based PCB"
+			(project "Ricardo-Cappy"
 				(path "/e4035b22-64c9-4a42-9837-ade8aec3882f/6c4172b2-a587-4406-930d-3d10d9850979"
 					(reference "Firing1")
@@
 		)
 		(instances
-			(project "Pi-based PCB"
+			(project "Ricardo-Cappy"
 				(path "/e4035b22-64c9-4a42-9837-ade8aec3882f/6c4172b2-a587-4406-930d-3d10d9850979"
 					(reference "R5")
@@
 		)
 		(instances
-			(project "Pi-based PCB"
+			(project "Ricardo-Cappy"
 				(path "/e4035b22-64c9-4a42-9837-ade8aec3882f/6c4172b2-a587-4406-930d-3d10d9850979"
 					(reference "R4")
@@
 		)
 		(instances
-			(project "Pi-based PCB"
+			(project "Ricardo-Cappy"
 				(path "/e4035b22-64c9-4a42-9837-ade8aec3882f/6c4172b2-a587-4406-930d-3d10d9850979"
 					(reference "#PWR027")
@@
 		)
 		(instances
-			(project "Pi-based PCB"
+			(project "Ricardo-Cappy"
 				(path "/e4035b22-64c9-4a42-9837-ade8aec3882f/6c4172b2-a587-4406-930d-3d10d9850979"
 					(reference "J6")
@@
 		)
 		(instances
-			(project "Pi-based PCB"
+			(project "Ricardo-Cappy"
 				(path "/e4035b22-64c9-4a42-9837-ade8aec3882f/6c4172b2-a587-4406-930d-3d10d9850979"
 					(reference "Q2")
@@
 		)
 		(instances
-			(project "Pi-based PCB"
+			(project "Ricardo-Cappy"
 				(path "/e4035b22-64c9-4a42-9837-ade8aec3882f/6c4172b2-a587-4406-930d-3d10d9850979"
 					(reference "D1")
@@
 		)
 		(instances
-			(project "Pi-based PCB"
+			(project "Ricardo-Cappy"
 				(path "/e4035b22-64c9-4a42-9837-ade8aec3882f/6c4172b2-a587-4406-930d-3d10d9850979"
 					(reference "#PWR09")
@@
 		)
 		(instances
-			(project "Pi-based PCB"
+			(project "Ricardo-Cappy"
 				(path "/e4035b22-64c9-4a42-9837-ade8aec3882f/6c4172b2-a587-4406-930d-3d10d9850979"
 					(reference "D16")
@@
 		)
 		(instances
-			(project "Pi-based PCB"
+			(project "Ricardo-Cappy"
 				(path "/e4035b22-64c9-4a42-9837-ade8aec3882f/6c4172b2-a587-4406-930d-3d10d9850979"
 					(reference "U6")
@@
 		)
 		(instances
-			(project "Pi-based PCB"
+			(project "Ricardo-Cappy"
 				(path "/e4035b22-64c9-4a42-9837-ade8aec3882f/6c4172b2-a587-4406-930d-3d10d9850979"
 					(reference "J4")
@@
 		)
 		(instances
-			(project "Pi-based PCB"
+			(project "Ricardo-Cappy"
 				(path "/e4035b22-64c9-4a42-9837-ade8aec3882f/6c4172b2-a587-4406-930d-3d10d9850979"
 					(reference "D5")
@@
 		)
 		(instances
-			(project "Pi-based PCB"
+			(project "Ricardo-Cappy"
 				(path "/e4035b22-64c9-4a42-9837-ade8aec3882f/6c4172b2-a587-4406-930d-3d10d9850979"
 					(reference "R20")
@@
 		)
 		(instances
-			(project "Pi-based PCB"
+			(project "Ricardo-Cappy"
 				(path "/e4035b22-64c9-4a42-9837-ade8aec3882f/6c4172b2-a587-4406-930d-3d10d9850979"
 					(reference "D2")
@@
 		)
 		(instances
-			(project "Pi-based PCB"
+			(project "Ricardo-Cappy"
 				(path "/e4035b22-64c9-4a42-9837-ade8aec3882f/6c4172b2-a587-4406-930d-3d10d9850979"
 					(reference "#PWR028")
@@
 		)
 		(instances
-			(project "Pi-based PCB"
+			(project "Ricardo-Cappy"
 				(path "/e4035b22-64c9-4a42-9837-ade8aec3882f/6c4172b2-a587-4406-930d-3d10d9850979"
 					(reference "Firing2")
@@
 		)
 		(instances
-			(project "Pi-based PCB"
+			(project "Ricardo-Cappy"
 				(path "/e4035b22-64c9-4a42-9837-ade8aec3882f/6c4172b2-a587-4406-930d-3d10d9850979"
 					(reference "D11")
@@
 		)
 		(instances
-			(project "Pi-based PCB"
+			(project "Ricardo-Cappy"
 				(path "/e4035b22-64c9-4a42-9837-ade8aec3882f/6c4172b2-a587-4406-930d-3d10d9850979"
 					(reference "D4")
@@
 		)
 		(instances
-			(project "Pi-based PCB"
+			(project "Ricardo-Cappy"
 				(path "/e4035b22-64c9-4a42-9837-ade8aec3882f/6c4172b2-a587-4406-930d-3d10d9850979"
 					(reference "R18")
@@
 		)
 		(instances
-			(project "Pi-based PCB"
+			(project "Ricardo-Cappy"
 				(path "/e4035b22-64c9-4a42-9837-ade8aec3882f/6c4172b2-a587-4406-930d-3d10d9850979"
 					(reference "U9")
@@
 		)
 		(instances
-			(project "Pi-based PCB"
+			(project "Ricardo-Cappy"
 				(path "/e4035b22-64c9-4a42-9837-ade8aec3882f/6c4172b2-a587-4406-930d-3d10d9850979"
 					(reference "#PWR013")
@@
 		)
 		(instances
-			(project "Pi-based PCB"
+			(project "Ricardo-Cappy"
 				(path "/e4035b22-64c9-4a42-9837-ade8aec3882f/6c4172b2-a587-4406-930d-3d10d9850979"
 					(reference "#PWR054")
@@
 		)
 		(instances
-			(project "Pi-based PCB"
+			(project "Ricardo-Cappy"
 				(path "/e4035b22-64c9-4a42-9837-ade8aec3882f/6c4172b2-a587-4406-930d-3d10d9850979"
 					(reference "#PWR019")
@@
 		)
 		(instances
-			(project "Pi-based PCB"
+			(project "Ricardo-Cappy"
 				(path "/e4035b22-64c9-4a42-9837-ade8aec3882f/6c4172b2-a587-4406-930d-3d10d9850979"
 					(reference "Q1")
@@
 		)
 		(instances
-			(project "Pi-based PCB"
+			(project "Ricardo-Cappy"
 				(path "/e4035b22-64c9-4a42-9837-ade8aec3882f/6c4172b2-a587-4406-930d-3d10d9850979"
 					(reference "#PWR025")
@@
 		)
 		(instances
-			(project "Pi-based PCB"
+			(project "Ricardo-Cappy"
 				(path "/e4035b22-64c9-4a42-9837-ade8aec3882f/6c4172b2-a587-4406-930d-3d10d9850979"
 					(reference "#PWR030")
@@
 		)
 		(instances
-			(project "Pi-based PCB"
+			(project "Ricardo-Cappy"
 				(path "/e4035b22-64c9-4a42-9837-ade8aec3882f/6c4172b2-a587-4406-930d-3d10d9850979"
 					(reference "D7")
@@
 		)
 		(instances
-			(project "Pi-based PCB"
+			(project "Ricardo-Cappy"
 				(path "/e4035b22-64c9-4a42-9837-ade8aec3882f/6c4172b2-a587-4406-930d-3d10d9850979"
 					(reference "#PWR056")

Commit message: Fixed power
Parts:
- removed J4, J6: Conn_01x02_Male, TerminalBlock_Phoenix:TerminalBlock_Phoenix_PT-1,5-2-3.5-H_1x02_P3.50mm_Horizontal, symbol Connector:Conn_01x02_Male
- added TC2: PYRO_1_OUT, Connector_Molex:Molex_Nano-Fit_105313-xx02_1x02_P2.50mm_Horizontal, symbol Device:Thermocouple
- added TC3: PYRO_2_OUT, Connector_Molex:Molex_Nano-Fit_105313-xx02_1x02_P2.50mm_Horizontal, symbol Device:Thermocouple
Connections:
- net DeployPWR: now also TC2.1 (+), TC3.1 (+)
- net at D2.2 (A), D4.1 (A), D4.2 (A)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: now also TC3.2 (-)
- net at D1.1 (A), D1.2 (A), D16.2 (A)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: now also TC2.2 (-)
Changed lines of the file:
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@@
+	(wire
+		(pts
+			(xy 138.43 13.97) (xy 130.81 13.97)
+		)
+		(stroke
+			(width 0)
+			(type default)
+		)
+	)
+	(wire
+		(pts
+			(xy 132.08 92.71) (xy 127 92.71)
+		)
+		(stroke
+			(width 0)
+			(type default)
+		)
+	)
 	(wire
 		(pts
@@
 	(wire
 		(pts
+			(xy 132.08 99.06) (xy 132.08 92.71)
+		)
+		(stroke
+			(width 0)
+			(type default)
+		)
+	)
+	(wire
+		(pts
 			(xy 138.43 48.26) (xy 138.43 55.88)
 		)
@@
 	(wire
 		(pts
+			(xy 135.89 19.05) (xy 130.81 19.05)
+		)
+		(stroke
+			(width 0)
+			(type default)
+		)
+	)
+	(wire
+		(pts
 			(xy 172.72 139.7) (xy 180.34 139.7)
 		)
@@
 	(wire
 		(pts
+			(xy 135.89 25.4) (xy 135.89 19.05)
+		)
+		(stroke
+			(width 0)
+			(type default)
+		)
+	)
+	(wire
+		(pts
 			(xy 137.16 99.06) (xy 142.24 99.06)
 		)
@@
 	(wire
 		(pts
+			(xy 138.43 25.4) (xy 138.43 13.97)
+		)
+		(stroke
+			(width 0)
+			(type default)
+		)
+	)
+	(wire
+		(pts
 			(xy 132.08 77.47) (xy 134.62 77.47)
 		)
@@
 	(wire
 		(pts
+			(xy 134.62 99.06) (xy 134.62 87.63)
+		)
+		(stroke
+			(width 0)
+			(type default)
+		)
+	)
+	(wire
+		(pts
 			(xy 137.16 104.14) (xy 135.89 104.14)
+		)
+		(stroke
+			(width 0)
+			(type default)
+		)
+	)
+	(wire
+		(pts
+			(xy 134.62 87.63) (xy 127 87.63)
 		)
 		(stroke
@@
 				(path "/e4035b22-64c9-4a42-9837-ade8aec3882f/6c4172b2-a587-4406-930d-3d10d9850979"
 					(reference "#PWR027")
-					(unit 1)
-				)
-			)
-		)
-	)
-	(symbol
-		(lib_id "Connector:Conn_01x02_Male")
-		(at 132.08 93.98 90)
-		(mirror x)
-		(unit 1)
-		(exclude_from_sim no)
-		(in_bom yes)
-		(on_board yes)
-		(dnp no)
-		(property "Reference" "J6"
-			(at 131.2418 93.7803 90)
-			(effects
-				(font
-					(size 1.27 1.27)
-				)
-				(justify left)
-			)
-		)
-		(property "Value" "Conn_01x02_Male"
-			(at 131.2418 96.3172 90)
-			(effects
-				(font
-					(size 1.27 1.27)
-				)
-				(justify left)
-			)
-		)
-		(property "Footprint" "TerminalBlock_Phoenix:TerminalBlock_Phoenix_PT-1,5-2-3.5-H_1x02_P3.50mm_Horizontal"
-			(at 132.08 93.98 0)
-			(effects
-				(font
-					(size 1.27 1.27)
-				)
-				(hide yes)
-			)
-		)
-		(property "Datasheet" "~"
-			(at 132.08 93.98 0)
-			(effects
-				(font
-					(size 1.27 1.27)
-				)
-				(hide yes)
-			)
-		)
-		(property "Description" ""
-			(at 132.08 93.98 0)
-			(effects
-				(font
-					(size 1.27 1.27)
-				)
-				(hide yes)
-			)
-		)
-		(pin "1"
-		)
-		(pin "2"
-		)
-		(instances
-			(project "Ricardo-Cappy"
-				(path "/e4035b22-64c9-4a42-9837-ade8aec3882f/6c4172b2-a587-4406-930d-3d10d9850979"
-					(reference "J6")
 					(unit 1)
 				)
@@
 	)
 	(symbol
-		(lib_id "Connector:Conn_01x02_Male")
-		(at 135.89 20.32 90)
-		(mirror x)
-		(unit 1)
-		(exclude_from_sim no)
-		(in_bom yes)
-		(on_board yes)
-		(dnp no)
-		(property "Reference" "J4"
-			(at 135.0518 20.1203 90)
-			(effects
-				(font
-					(size 1.27 1.27)
-				)
-				(justify left)
-			)
-		)
-		(property "Value" "Conn_01x02_Male"
-			(at 135.0518 22.6572 90)
-			(effects
-				(font
-					(size 1.27 1.27)
-				)
-				(justify left)
-			)
-		)
-		(property "Footprint" "TerminalBlock_Phoenix:TerminalBlock_Phoenix_PT-1,5-2-3.5-H_1x02_P3.50mm_Horizontal"
-			(at 135.89 20.32 0)
-			(effects
-				(font
-					(size 1.27 1.27)
-				)
-				(hide yes)
-			)
-		)
-		(property "Datasheet" "~"
-			(at 135.89 20.32 0)
-			(effects
-				(font
-					(size 1.27 1.27)
-				)
-				(hide yes)
-			)
-		)
-		(property "Description" ""
-			(at 135.89 20.32 0)
-			(effects
-				(font
-					(size 1.27 1.27)
-				)
-				(hide yes)
-			)
-		)
-		(pin "1"
-		)
-		(pin "2"
-		)
-		(instances
-			(project "Ricardo-Cappy"
-				(path "/e4035b22-64c9-4a42-9837-ade8aec3882f/6c4172b2-a587-4406-930d-3d10d9850979"
-					(reference "J4")
-					(unit 1)
-				)
-			)
-		)
-	)
-	(symbol
 		(lib_id "Device:LED")
 		(at 168.91 59.69 90)
@@
 				(path "/e4035b22-64c9-4a42-9837-ade8aec3882f/6c4172b2-a587-4406-930d-3d10d9850979"
 					(reference "R18")
+					(unit 1)
+				)
+			)
+		)
+	)
+	(symbol
+		(lib_id "Device:Thermocouple")
+		(at 133.35 16.51 180)
+		(unit 1)
+		(exclude_from_sim no)
+		(in_bom yes)
+		(on_board yes)
+		(dnp no)
+		(property "Reference" "TC2"
+			(at 134.0358 24.765 0)
+			(effects
+				(font
+					(size 1.27 1.27)
+				)
+			)
+		)
+		(property "Value" "PYRO_1_OUT"
+			(at 134.0358 22.4536 0)
+			(effects
+				(font
+					(size 1.27 1.27)
+				)
+			)
+		)
+		(property "Footprint" "Connector_Molex:Molex_Nano-Fit_105313-xx02_1x02_P2.50mm_Horizontal"
+			(at 147.955 17.78 0)
+			(effects
+				(font
+					(size 1.27 1.27)
+				)
+				(hide yes)
+			)
+		)
+		(property "Datasheet" "~"
+			(at 147.955 17.78 0)
+			(effects
+				(font
+					(size 1.27 1.27)
+				)
+				(hide yes)
+			)
+		)
+		(property "Description" ""
+			(at 133.35 16.51 0)
+			(effects
+				(font
+					(size 1.27 1.27)
+				)
+				(hide yes)
+			)
+		)
+		(pin "1"
+		)
+		(pin "2"
+		)
+		(instances
+			(project "Ricardo-Cappy"
+				(path "/e4035b22-64c9-4a42-9837-ade8aec3882f/6c4172b2-a587-4406-930d-3d10d9850979"
+					(reference "TC2")
 					(unit 1)
 				)
@@
 					(unit 1)
 				)
+			)
+		)
+	)
+	(symbol
+		(lib_id "Device:Thermocouple")
+		(at 129.54 90.17 180)
+		(unit 1)
+		(exclude_from_sim no)
+		(in_bom yes)
+		(on_board yes)
+		(dnp no)
+		(property "Reference" "TC3"
+			(at 130.2258 98.425 0)
+			(effects
+				(font
+					(size 1.27 1.27)
+				)
+			)
+		)
+		(property "Value" "PYRO_2_OUT"
+			(at 130.2258 96.1136 0)
+			(effects
+				(font
+					(size 1.27 1.27)
+				)
+			)
+		)
+		(property "Footprint" "Connector_Molex:Molex_Nano-Fit_105313-xx02_1x02_P2.50mm_Horizontal"
+			(at 144.145 91.44 0)
+			(effects
+				(font
+					(size 1.27 1.27)
+				)
+				(hide yes)
+			)
+		)
+		(property "Datasheet" "~"
+			(at 144.145 91.44 0)
+			(effects
+				(font
+					(size 1.27 1.27)
+				)
+				(hide yes)
+			)
+		)
+		(property "Description" ""
+			(at 129.54 90.17 0)
+			(effects
+				(font
+					(size 1.27 1.27)
+				)
+				(hide yes)
+			)
+		)
+		(pin "1"
+		)
+		(pin "2"
+		)
+		(instances
+			(project "Ricardo-Cappy"
+				(path "/e4035b22-64c9-4a42-9837-ade8aec3882f/6c4172b2-a587-4406-930d-3d10d9850979"
+					(reference "TC3")
+					(unit 1)
+				)
